File: VLT.kicad_sch (KiCad schematic)
At the start: 95 parts, among them J1 TFT, J2 DEBUG, J3 FPC_4P_0.5mm, J4 LED_EXP, J5 Conn_01x04_MountingPin, J6 TFT, Q1 AO3401A, Q2 BSS138, Q3 AO3401A, Q4 BSS138, SW1 SW_Push_Momentary, U1 AP2112K-3.3, U2 W25Q128JVS, U3 RP2350B-QFN80, U4 MPR121QR2, Y1 12MHz

Commit message: PCB rev1 done — schematic/layout updates, drop stale production exports
- Schematic + PCB updates across VLT.kicad_pcb/sch, leds.kicad_sch, sensors.kicad_sch
- Remove production/ rev1 exports (zip/bom/positions/netlist) — regenerated on demand
- Drop fabrication-toolkit-options.json (not used)
- gitignore VLT+Dev/ experimental layouts
Parts:
- removed C1, C10, C11, C12, C17, C2, C27, C3, C4, C5, C6, C7, C8, C9: 100nF, Mars_Library:C_0402, symbol Mars_Library:C_0402
- removed C18: 10uF, Mars_Library:C_0402, symbol Mars_Library:C_0402
- removed C19: 4.7uF, Mars_Library:C_0402, symbol Mars_Library:Capacitor_0402_4.7uF
- removed C20, C21: 4.7uF, Mars_Library:C_0402, symbol Mars_Library:C_0603
- removed C25, C26: 30pF, Mars_Library:C_0402, symbol Mars_Library:C_0402
- removed J3: FPC_4P_0.5mm, Mars_Library:XUNPU_FPC-05F-4PH20_1x4-1MP_P0.5mm, symbol Mars_Library:FPC_4P_0.5mm
- removed J5: Conn_01x04_MountingPin, Connector_JST:JST_SH_SM04B-SRSS-TB_1x04-1MP_P1.00mm_Horizontal, symbol Connector_Generic_MountingPin:Conn_01x04_MountingPin
- removed J6: TFT, Mars_Library:XUNPU_FPC-05F-12PH20_1x12-1MP_P0.5mm, symbol Mars_Library:Conn_FPC_12P_0.5mm_MP
- removed L1: 3.3uH, Inductor_SMD:L_Murata_DFE201610P, symbol Device:L
- removed R1: 33R, Mars_Library:R_0402, symbol Mars_Library:R_0402
- removed R10: 1K, Mars_Library:R_0402, symbol Mars_Library:R_0402
- removed R2, R3: 27R, Mars_Library:R_0402, symbol Mars_Library:R_0402
- removed R30, R31, R32, R33: 10K, Mars_Library:R_0402, symbol Mars_Library:Resistor_R_0402_10K
- removed S1: RKJXT1F42001, RKJXT1F42001:XDCR_RKJXT1F42001, symbol RKJXT1F42001:RKJXT1F42001
- removed SW1: SW_Push_Momentary, Mars_Library:SW_2x3x0.65mm_SPST_Tiny, symbol Mars_Library:SW_Push_Momentary
- removed TP1: GP0, Mars_Library:TestPoint_Pad_D1.0mm_Minimal, symbol PCM_4ms_Connector:TestPoint
- removed TP2: GP1, Mars_Library:TestPoint_Pad_D1.0mm_Minimal, symbol PCM_4ms_Connector:TestPoint
- removed TP3: BOOT, Mars_Library:TestPoint_Pad_D1.0mm_Minimal, symbol PCM_4ms_Connector:TestPoint
- removed TP4: GND, Mars_Library:TestPoint_Pad_D1.0mm_Minimal, symbol PCM_4ms_Connector:TestPoint
- removed U3: RP2350B-QFN80, RP2350_KiCad:RP2350B_QFN-80_EP_10.573x10.573_Pitch0.4mm, symbol rp2350b-qfn80:RP2350B-QFN80
- removed Y1: 12MHz, Crystal:Crystal_SMD_SeikoEpson_TSX3225-4Pin_3.2x2.5mm, symbol Device:Crystal_GND24
- added C1, C10, C11, C12, C17, C2, C27, C3, C31, C32, C6, C7, C8, C9: 100nF, Mars_Library:C_0402, symbol Mars_Library:Capacitor_C_0603_100nF_0.1uF
- added C18, C21, C4, C5: 20pF, Mars_Library:C_0402, symbol Mars_Library:Capacitor_C_0402
- added C19, C33: 100nF, Mars_Library:C_0402, symbol Mars_Library:C_0402
- added C20, C34: 1uF, Mars_Library:C_0402, symbol Mars_Library:C_0402
- added C25, C26: 4.7uF, Mars_Library:C_0402, symbol Mars_Library:Capacitor_C_0402_4.7uF
- added C35, C36: 10uF, Mars_Library:C_0402, symbol Mars_Library:C_0402
- added FB2: 60R, Mars_Library:Ferrite_0402, symbol Mars_Library:FerriteBead_0805
- added J3: MPR_ELE, Mars_Library:XUNPU_FPC-05F-12PH20_1x12-1MP_P0.5mm, symbol Connector_Generic_MountingPin:Conn_01x12_MountingPin
- added J5: CTP, Mars_Library:XUNPU_FPC-05F-6PH20_1x6-1MP_P0.5mm, symbol Connector_Generic_MountingPin:Conn_01x06_MountingPin
- added J6: UART, Connector_JST:JST_SH_SM02B-SRSS-TB_1x02-1MP_P1.00mm_Horizontal, symbol Connector_Generic_MountingPin:Conn_01x02_MountingPin
- added J7: DEBUG, Connector_JST:JST_SH_SM06B-SRSS-TB_1x06-1MP_P1.00mm_Horizontal, symbol Connector_Generic_MountingPin:Conn_01x06_MountingPin
- added Q5: AO3401A, PCM_4ms_Package_SOT:SOT-23, symbol Transistor_FET:AO3401A
- added R1, R2: 10K, Mars_Library:R_0402, symbol Mars_Library:Resistor_R_0603
- added R10: 12K, Mars_Library:R_0402, symbol Mars_Library:Resistor_R_0603
- added R3: 0R, Mars_Library:R_0402, symbol Mars_Library:Resistor_R_0402_100R
- added R30, R31, R32, R33, R34, R35: 22R, Mars_Library:R_0402, symbol Mars_Library:R_0603
- added S1: BOOT, B3U-1000P:SW_B3U-1000P, symbol B3U-1000P:B3U-1000P
- added TP1: TX, Mars_Library:TestPoint_Pad_D1.0mm_Minimal, symbol Connector:TestPoint
- added TP2: RX, Mars_Library:TestPoint_Pad_D1.0mm_Minimal, symbol Connector:TestPoint
- added TP3: NRST, Mars_Library:TestPoint_Pad_D1.0mm_Minimal, symbol Connector:TestPoint
- added TP4: BOOT, Mars_Library:TestPoint_Pad_D1.0mm_Minimal, symbol Connector:TestPoint
- added TP5: GND, Mars_Library:TestPoint_Pad_D1.0mm_Minimal, symbol Connector:TestPoint
- added U3: STM32H723VGTx, Package_QFP:LQFP-100_14x14mm_P0.5mm, symbol MCU_ST_STM32H7:STM32H723VGTx
- added U5: USB3300-EZK, Package_DFN_QFN:QFN-32-1EP_5x5mm_P0.5mm_EP3.45x3.45mm, symbol Interface_USB:USB3300-EZK
- added U6: W25Q32JVZP, Package_SON:WSON-8-1EP_6x5mm_P1.27mm_EP3.4x4.3mm, symbol Memory_Flash:W25Q32JVZP
- added U7: (no value), Mars_Library:XUNPU_FPC-05F-12PH20_1x12-1MP_P0.5mm, symbol Mars_Library:TouchDisplay
- added Y1: 24MHz, Crystal:Crystal_SMD_3225-4Pin_3.2x2.5mm, symbol Device:Crystal_GND24_Small
- added Y2: 25MHz, Crystal:Crystal_SMD_3225-4Pin_3.2x2.5mm, symbol Device:Crystal_GND24_Small
- FB1: footprint Mars_Library:Ferrite_0603 -> Mars_Library:Ferrite_0805
- FB3: value 600R -> 60R
- J2: footprint Mars_Library:SWD_Debug_PinHeader_1x04_P2.54mm -> Mars_Library:SWD_Debug_PinHeader_1x05_P2.54mm; symbol Mars_Library:SWD_Header_4P -> Mars_Library:SWD_Header_5P; now in the parts list
- R29, TH1: now fitted
- R6, R8: value 27R -> 22R
Connections:
- net +3V3: now also C10.1, C11.1, C12.1, C17.1, C32.1, C6.1, C7.1, C8.1, C9.1, J5.6 (Pin_6), J7.5 (Pin_5), S1.1, U3.100 (VDD), U3.11 (VDD), U3.27 (VDD), U3.50 (VDD), U3.6 (VBAT), U3.75 (VDD), U5.16 (VDD3.3), U5.25 (VDD3.3), U5.30 (VDD3.3), U5.31 (REG_EN), U5.6 (VDD3.3), U6.8 (VCC), U7.7 (VCC)
- net +3V3A: now also C19.2, C20.2, C36.2, FB2.1, U3.21 (VDDA)
- net +5V: now also C3.1, J7.6 (Pin_6), Q5.2 (S), R1.1
- net +5V_LED: now also Q5.3 (D)
- net ADC1: now also U3.22 (PA0)
- net ADC2: now also U3.23 (PA1)
- net ADC3: now also U3.24 (PA2)
- net ADC4: now also U3.28 (PA4)
- net ADC5: now also U3.30 (PA6)
- net ADC6: now also U3.32 (PC4)
- net D+: now also U5.7 (DP)
- net D-: now also U5.8 (DM)
- net ELE0: now also J3.1 (Pin_1)
- net ELE1: now also J3.2 (Pin_2)
- net ELE10: now also J3.11 (Pin_11)
- net ELE11: now also J3.12 (Pin_12)
- net ELE2: now also J3.3 (Pin_3)
- net ELE3: now also J3.4 (Pin_4)
- net ELE4: now also J3.5 (Pin_5)
- net ELE5: now also J3.6 (Pin_6)
- net ELE6: now also J3.7 (Pin_7)
- net ELE7: now also J3.8 (Pin_8)
- net ELE8: now also J3.9 (Pin_9)
- net ELE9: now also J3.10 (Pin_10)
- net ENC_A: now also ENC1.B, U3.64 (PC7); no longer ENC1.A
- net ENC_B: now also ENC1.A, U3.63 (PC6); no longer ENC1.B
- net ENC_SW: now also ENC1.S2, U3.67 (PA8); no longer ENC1.S1
- net GND: now also ENC1.S1, SD1.SH1 (SHIELD), C1.2, C10.2, C11.2, C12.2, C17.2, C18.1, C19.1, C2.2, C20.1, C21.1, C25.2, C26.2, C27.1, C3.2, C31.2, C32.2, C33.1, C34.1, C35.1, C36.1, C4.1, C5.1, C6.2, C7.2, C8.2, C9.2, J3.MP (MountPin), J5.5 (Pin_5), J5.MP (MountPin), J6.MP (MountPin), J7.1 (Pin_1), J7.MP (MountPin), R10.1, R2.1, TP5.1, U3.10 (VSS), U3.19 (VSSA), U3.26 (VSS), U3.49 (VSS), U3.74 (VSS), U3.99 (VSS), U5.1 (GND), U5.2 (GND), U5.33 (GND), U6.4 (GND), U6.9 (EP), U7.2 (GND), U7.MP, Y1.2, Y1.4, Y2.2, Y2.4; no longer ENC1.S2
- net LED:N_DRAIN/P_GATE: now also Q5.1 (G)
- net MPR_IRQ: now also U3.93 (PB7)
- net NTC: now also U3.16 (PC1)
- net SD_CLK: now also R32.1, U3.80 (PC12); no longer SD1.5 (CLK)
- net SWCLK: now also J7.4 (Pin_4), U3.76 (PA14(JTCK)
- net SWDIO: now also J7.3 (Pin_3), U3.72 (PA13(JTMS)
- net TFT_BL: now also U7.1 (LEDA)
- net TFT_CLK: now also U7.6 (TFT_CLK)
- net TFT_CS: now also U3.39 (PE9), U7.8 (TFT_CS)
- net TFT_DC: now also U3.40 (PE10), U7.4 (TFT_DC)
- net TFT_MOSI: now also U7.5 (TFT_MOSI)
- net TFT_RES: now also U3.38 (PE8), U7.3 (TFT_RST)
- net R:E12: now reaches R6.1
- net R:E12: now also U3.42 (PE12)
- net R:E14: now reaches R8.1
- net R:E14: now also U3.44 (PE14)
- net S.D2: now reaches SD1.1 (DAT2)
- net S.D2: now also R35.1
- net S.D1: now reaches SD1.8 (DAT1)
- net S.D1: now also R34.1
- net CARD_DETECT renamed SD_CARD
- net SD_CARD: now also U3.7 (PC13)
- net COM1 renamed MUX_COM1
- net COM2 renamed MUX_COM2
- net COM3 renamed MUX_COM3
- net COM4 renamed MUX_COM4
- net COM5 renamed MUX_COM5
- net COM6 renamed MUX_COM6
- net GP21_ERM_GATE renamed ERM_GATE
- net ERM_GATE: now also U3.71 (PA12)
- net GP29_LED_EN renamed RGB_GATE
- net RGB_GATE: now also U3.3 (PE4)
- net LED_EXP renamed WS2812_DOUT
- net LED_GATE renamed LED:R>GATE
- net MPR_SCL renamed I2C1_SCL
- net I2C1_SCL: now also J5.4 (Pin_4), U3.95 (PB8), U7.12 (CTP_SCL)
- net MPR_SDA renamed I2C1_SDA
- net I2C1_SDA: now also J5.3 (Pin_3), U3.96 (PB9), U7.11 (CTP_SDA)
- net PWM_TFT_BL renamed TFT_BL_GATE
- net TFT_BL_GATE: now also U3.43 (PE13)
- net QSPI_SCLK renamed QSPI_CLK
- net QSPI_CLK: now also U3.36 (PB2), U6.6 (CLK)
- net QSPI_SD0 renamed QSPI_IO0
- net QSPI_IO0: now also U3.58 (PD11), U6.5 (DI/IO_{0})
- net QSPI_SD1 renamed QSPI_IO1
- net QSPI_IO1: now also U3.59 (PD12), U6.2 (DO/IO_{1})
- net QSPI_SD2 renamed QSPI_IO2
- net QSPI_IO2: now also U3.1 (PE2), U6.3 (~{WP}/IO_{2})
- net QSPI_SD3 renamed QSPI_IO3
- net QSPI_IO3: now also U3.60 (PD13), U6.7 (~{HOLD}/~{RESET}/IO_{3})
- net QSPI_SS renamed QSPI_CS
- net QSPI_CS: now also U3.41 (PE11), U6.1 (~{CS})
- net SD_CS renamed S.D3
- net S.D3: now also R30.2
- net SD_MISO renamed S.D0
- net S.D0: now also R33.2
- net SD_MOSI renamed S.CMD
- net S.CMD: now also R31.2
- new net: R10.2, U5.32 (RBIAS)
- new net: R3.2, U3.55 (PD8)
- new net: R1.2, U5.4 (VBUS)
- new net: C25.1, U3.48 (VCAP)
- new net: C26.1, U3.73 (VCAP)
- new net +1V8A_USB: C1.1, U5.29 (VDDA1.8)
- new net +1V8_USB: C2.1, C31.1, U5.15 (VDD1.8), U5.26 (VDD1.8)
- new net BOOT: R2.2, S1.2, TP4.1, U3.94 (BOOT0)
- new net CTP_INT: J5.1 (Pin_1), U3.54 (PB15), U7.9 (CTP_INT)
- new net CTP_RST: J5.2 (Pin_2), U3.53 (PB14), U7.10 (CTP_RST)
- new net HSE_IN: C18.2, U3.12 (PH0), Y2.1
- new net HSE_OUT: C21.2, U3.13 (PH1), Y2.3
- new net MUX_S0: U3.85 (PD4)
- new net MUX_S1: U3.86 (PD5)
- new net MUX_S2: U3.87 (PD6)
- new net MUX_S3: U3.88 (PD7)
- new net NRST: C27.2, J2.5 (Pin_5), J7.2 (Pin_2), TP3.1, U3.14 (NRST)
- new net S.CLK: R32.2, SD1.5 (CLK)
- new net SD_CMD: R31.1, U3.83 (PD2)
- new net SD_D0: R33.1, U3.65 (PC8)
- new net SD_D1: R34.2, U3.66 (PC9)
- new net SD_D2: R35.2, U3.78 (PC10)
- new net SD_D3: R30.1, U3.79 (PC11)
- new net UART_RX: J6.2 (Pin_2), TP2.1, U3.69 (PA10)
- new net UART_TX: J6.1 (Pin_1), TP1.1, U3.68 (PA9)
- new net ULPI_CLK: U3.29 (PA5), U5.14 (CLKOUT)
- new net ULPI_D0: U3.25 (PA3), U5.24 (DATA0)
- new net ULPI_D1: U3.34 (PB0), U5.23 (DATA1)
- new net ULPI_D2: U3.35 (PB1), U5.22 (DATA2)
- new net ULPI_D3: U3.46 (PB10), U5.21 (DATA3)
- new net ULPI_D4: U3.47 (PB11), U5.20 (DATA4)
- new net ULPI_D5: U3.51 (PB12), U5.19 (DATA5)
- new net ULPI_D6: U3.52 (PB13), U5.18 (DATA6)
- new net ULPI_D7: U3.91 (PB5), U5.17 (DATA7)
- new net ULPI_DIR: U3.17 (PC2_C), U5.12 (DIR)
- new net ULPI_NXT: U3.18 (PC3_C), U5.11 (NXT)
- new net ULPI_RST: R3.1, U5.9 (RESET)
- new net ULPI_STP: U3.15 (PC0), U5.13 (STP)
- new net VREF+: C33.2, C34.2, C35.2, FB2.2, U3.20 (VREF+)
- new net WS2812_DIN: U3.31 (PA7)
- new net XI: C4.2, U5.28 (XI), Y1.3
- new net XO: C5.2, U5.27 (XO), Y1.1
- no-connect marks 2 -> 3
Other:
- sheet leds ports: added WS2812_DIN, WS2812_DOUT; removed none
- sheet sensors ports: added COM1, COM2, COM3, COM4, COM5, COM6, S0, S1, S2, S3; removed none
- note added: "81 key + 4, 10 ambient, 3 status = 98 LEDs total"
- note added: "Debug + headers"
- note removed: "81 key, 10 ambient, 3 status = 94 LEDs total"
- note removed: "Debug + flash headers"
- moved on the sheet: C15, C22, C23, C24, C29, D1, ENC1, ERM1, FB3, FID1, FID2, FID3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
